File: hw/driver_22mm/Driver.kicad_sch (KiCad schematic)
At the start: 51 parts, among them J1 +LED, J10 R, J11 G, J12 Button, J13 Button_GND, J2 -LED, J3 Button LED, J4 Button LED GND, J5 SWDIO, J6 SWCLK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

Commit message: Driver v2 changes
Parts:
- added R5: 7m - R_SENSE_MAIN, Resistor_SMD_AKL:R_0805_2012Metric, symbol PCM_Resistor_AKL:R_0402
- added U5: XS3A1T3157GSH, XSON6_SOT1202_NEX, symbol XS3A1T3157GSH:XS3A1T3157GSH
- Q1: value 7m - R_SENSE_MAIN -> ~
- R13: value 2.25M - R_BAT_TOP -> 1.6M - R_BAT_TOP
- R3: value 254k - R_DAC_TOP -> 285k - R_DAC_TOP
- R6: footprint Resistor_SMD_AKL:R_0805_2012Metric -> Resistor_SMD_AKL:R_0402_1005Metric
- U4: value NCP114AMX250TCG -> NCP114AMX280TCG
Connections:
- net -LED: now also U5.3 (Y1); no longer U2.3 (+)
- net GND: now also R5.2, U5.2 (GND); no longer Q1.4 (S)
- net VCC: now also U5.5 (VCC)
- net SHUNT_SELECT: now reaches U3.1 (PC14)
- net SHUNT_SELECT: now also U5.6 (S)
- net BOOST_EN: now reaches U3.28 (PB6)
- net BOOST_EN: now also R1.1
- net EN renamed OPAMP_EN
- net OPAMP_EN: no longer R1.1
- new net: Q1.4 (S), R5.1, U5.1 (Y2)
- new net: U2.3 (+), U5.4 (Z)
- no-connect marks 12 -> 10
Other:
- moved on the sheet: Q1, R6

Commit message: Stuff
Parts:
- removed J13: Button_GND, TestPoint:TestPoint_Pad_D1.0mm, symbol Connector_Generic:Conn_01x01
- J4: value Button LED GND -> Wire GND; footprint TestPoint:TestPoint_Pad_D1.0mm -> TestPoint:TestPoint_Pad_D1.0mm_copy
- R11: value 450k - R_FB_C -> 434k - R_FB_C
- R5: value 7m - R_SENSE_MAIN -> 10m - R_SENSE_MAIN
Changed lines of the file:
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@@
 	(symbol
 		(lib_id "Connector_Generic:Conn_01x01")
-		(at 266.7 217.17 180)
-		(unit 1)
-		(exclude_from_sim no)
-		(in_bom yes)
-		(on_board yes)
-		(dnp no)
-		(fields_autoplaced yes)
-		(property "Reference" "J13"
-			(at 266.7 210.82 0)
-			(effects
-				(font
-					(size 1.27 1.27)
-				)
-			)
-		)
-		(property "Value" "Button_GND"
-			(at 266.7 213.36 0)
-			(effects
-				(font
-					(size 1.27 1.27)
-				)
-			)
-		)
-		(property "Footprint" "TestPoint:TestPoint_Pad_D1.0mm"
-			(at 266.7 217.17 0)
-			(effects
-				(font
-					(size 1.27 1.27)
-				)
-				(hide yes)
-			)
-		)
-		(property "Datasheet" "~"
-			(at 266.7 217.17 0)
-			(effects
-				(font
-					(size 1.27 1.27)
-				)
-				(hide yes)
-			)
-		)
-		(property "Description" "Generic connector, single row, 01x01, script generated (kicad-library-utils/schlib/autogen/connector/)"
-			(at 266.7 217.17 0)
-			(effects
-				(font
-					(size 1.27 1.27)
-				)
-				(hide yes)
-			)
-		)
-		(pin "1"
-		)
-		(instances
-			(project "Driver"
-				(path "/7fa7dcf1-f7f2-431d-b0e2-843364aa27ee"
-					(reference "J13")
-					(unit 1)
-				)
-			)
-		)
-	)
-	(symbol
-		(lib_id "Connector_Generic:Conn_01x01")
 		(at 353.06 228.6 0)
 		(unit 1)
@@
 			)
 		)
-		(property "Value" "Button LED GND"
+		(property "Value" "Wire GND"
 			(at 266.7 223.52 0)
 			(effects
@@
 			)
 		)
-		(property "Footprint" "TestPoint:TestPoint_Pad_D1.0mm"
+		(property "Footprint" "TestPoint:TestPoint_Pad_D1.0mm_copy"
 			(at 266.7 227.33 0)
 			(effects
@@
 			)
 		)
-		(property "Value" "7m - R_SENSE_MAIN"
+		(property "Value" "10m - R_SENSE_MAIN"
 			(at 200.66 278.384 90)
 			(effects
@@
 			)
 		)
-		(property "Value" "450k - R_FB_C"
+		(property "Value" "434k - R_FB_C"
 			(at 185.42 193.04 90)
 			(effects
